File: ESP32_RemoteWetherstation/Hardware/ESP32_RemoteWetherstation/ESP32_RemoteWetherstation.kicad_sch (KiCad schematic)
At the start: 5 parts, among them J301 BOOT, J302 UART, U303 ESP32-S3-MINI-1

Commit message: Connected IO
Connections:
- net IO2: now reaches U303.6 (IO2)
Other:
- added sheet I_Sense (I_Sense.kicad_sch)
- note added: "I Sense"
Changed lines of the file:
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@@
+		)
+	)
+	(text "I Sense"
+		(exclude_from_sim no)
+		(at 156.718 97.282 0)
+		(effects
+			(font
+				(size 1.27 1.27)
+			)
 		)
 	)
@@
 	(polyline
 		(pts
+			(xy 194.31 95.25) (xy 194.31 114.3)
+		)
+		(stroke
+			(width 0)
+			(type dash)
+		)
+	)
+	(polyline
+		(pts
 			(xy 139.7 57.15) (xy 110.49 57.15)
 		)
@@
 	(wire
 		(pts
+			(xy 25.4 49.53) (xy 27.94 49.53)
+		)
+		(stroke
+			(width 0)
+			(type default)
+		)
+	)
+	(wire
+		(pts
 			(xy 81.28 39.37) (xy 85.09 39.37)
 		)
@@
 		)
 	)
+	(polyline
+		(pts
+			(xy 194.31 95.25) (xy 152.4 95.25)
+		)
+		(stroke
+			(width 0)
+			(type dash)
+		)
+	)
 	(wire
 		(pts
@@
 		)
 	)
+	(polyline
+		(pts
+			(xy 194.31 114.3) (xy 152.4 114.3)
+		)
+		(stroke
+			(width 0)
+			(type dash)
+		)
+	)
 	(global_label "SDA"
 		(shape input)
@@
 				)
 				(justify left)
+				(hide yes)
+			)
+		)
+	)
+	(global_label "IO2"
+		(shape input)
+		(at 25.4 49.53 180)
+		(fields_autoplaced yes)
+		(effects
+			(font
+				(size 1.27 1.27)
+			)
+			(justify right)
+		)
+		(property "Intersheetrefs" "${INTERSHEET_REFS}"
+			(at 19.27 49.53 0)
+			(effects
+				(font
+					(size 1.27 1.27)
+				)
+				(justify right)
 				(hide yes)
 			)
@@
 				)
 			)
+		)
+	)
+	(sheet
+		(at 153.67 100.33)
+		(size 12.7 3.81)
+		(exclude_from_sim no)
+		(in_bom yes)
+		(on_board yes)
+		(dnp no)
+		(fields_autoplaced yes)
+		(stroke
+			(width 0.1524)
+			(type solid)
+		)
+		(fill
+			(color 0 0 0 0.0000)
+		)
+		(property "Sheetname" "I_Sense"
+			(at 153.67 99.6184 0)
+			(effects
+				(font
+					(size 1.27 1.27)
+				)
+				(justify left bottom)
+			)
+		)
+		(property "Sheetfile" "I_Sense.kicad_sch"
+			(at 153.67 104.7246 0)
+			(effects
+				(font
+					(size 1.27 1.27)
+				)
+				(justify left top)
+			)
+		)
+		(instances
+			(project "ESP32_RemoteWetherstation"
+				(path "/bb194ab9-ddae-46dd-ae5d-1e0c862ad374"
+					(page "12")
+				)
+			)
