File: ESP32_RemoteWetherstation/Hardware/ESP32_RemoteWetherstation/ESP32_RemoteWetherstation.kicad_pcb (KiCad board)
At the start: 2 copper layers, 48.6 x 28.9 mm, 41 parts, among them IC301 AP2210K-3.3TRG1, J301 BOOT, J302 UART, J303 VCC, J304 GND, J305 OpenDrain, J306 OpenDrain, J307 OpenDrain, J308 OpenDrain, J310 Analog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

Commit message: approximately arranged components (#10)
Parts:
- C305, C306, C307, IC301, J310, J311, J312, Q301, Q302, Q303, Q304, R304, R305, R306, R307, R310, R311, R312, R313, R314, R315: moved to F.Cu
- J305, J306, J307, J308, NT301: moved to B.Cu
- moved J312 132.1 mm to (43.9, 136.0), turned to 0 degrees
- moved R314 131.1 mm to (46.5, 135.7), turned to -90 degrees
- moved R315 129.9 mm to (46.5, 138.8), turned to -90 degrees
- moved J310 129.5 mm to (43.9, 142.3), turned to 0 degrees
- moved R310 128.8 mm to (46.5, 142.0), turned to -90 degrees
- moved R311 127.8 mm to (46.5, 145.0), turned to -90 degrees
- moved J301 124.8 mm to (43.9, 102.4)
- moved J311 118.0 mm to (43.9, 129.7), turned to 0 degrees
- moved R312 117.0 mm to (46.5, 129.4), turned to -90 degrees
- moved R313 115.8 mm to (46.5, 132.4), turned to -90 degrees
- moved C304 114.1 mm to (53.1, 117.9), turned to 90 degrees
- moved J302 106.0 mm to (66.0, 105.1), turned to 0 degrees
- moved J304 105.8 mm to (58.1, 145.3), turned to 90 degrees
- moved C303 105.6 mm to (53.1, 133.4), turned to 90 degrees
- moved J303 104.7 mm to (53.1, 145.3), turned to 90 degrees
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Routing:
- net TXD0: track 28.2 -> 3.74 mm
- net +3V3: track 51.2 -> 72.1 mm, vias 3 -> 9
- net IO14: track 13.7 -> 0.00 mm, vias 1 -> 0
- net IO11: track 13.2 -> 1.45 mm, vias 1 -> 0
- net BOOT: track 13.0 -> 1.65 mm
- net IO17: track 10.8 -> 1.35 mm, vias 1 -> 0
- net IO12: track 7.12 -> 0.00 mm, vias 1 -> 0
- net IO15: track 6.80 -> 0.00 mm, vias 1 -> 0
- net IO13: track 4.18 -> 0.00 mm, vias 1 -> 0
- net VCC: track 0.00 -> 4.05 mm, vias 0 -> 1
- net RXD0: track 0.00 -> 3.76 mm
- net IO18: track 2.36 -> 1.36 mm, vias 1 -> 0
- net GND: track 16.0 -> 16.6 mm, vias 7 -> 8
- added copper zone on F.Cu, net +3V3
- added copper zone on F.Cu, net /IO/OpenDrainOutput/OpenDran
- added copper zone on F.Cu, net /IO/OpenDrainOutput1/OpenDran
- added copper zone on F.Cu, net /IO/OpenDrainOutput2/OpenDran
- added copper zone on F.Cu, net /IO/OpenDrainOutput3/OpenDran
- added copper zone on F.Cu, net IO12
- added copper zone on F.Cu, net IO13
- added copper zone on F.Cu, net IO14
- added copper zone on F.Cu, net IO15
- added copper zone on F.Cu, net VCC
- removed copper zone on B.Cu, net /IO/OpenDrainOutput/OpenDran
- removed copper zone on B.Cu, net /IO/OpenDrainOutput1/OpenDran
- removed copper zone on B.Cu, net /IO/OpenDrainOutput2/OpenDran
- removed copper zone on B.Cu, net /IO/OpenDrainOutput3/OpenDran
- removed copper zone on B.Cu, net IO12
- removed copper zone on B.Cu, net IO13
- removed copper zone on B.Cu, net IO14
- removed copper zone on B.Cu, net IO15
- removed copper zone on B.Cu, net VCC
Other:
- board size 48.6 x 28.9 mm -> 28.1 x 47.2 mm
- board text removed: "Mybe I need to change to 4 layer Gonna try switching the VCC to F.Cu, but not sure how this might help ToDo: Change VCC Layer, and check the price div. of 2-4 Layer PCB"

Commit message: placed all comps onesided (#11)
Parts:
- C301, C302, J305, J306, J307, J308, R301, R302, R303, RE_ESP301, U302: moved to F.Cu
- moved C302 15.0 mm to (42.8, 110.9), turned to 90 degrees
- moved R301 14.1 mm to (45.3, 112.8), turned to 180 degrees
- moved U302 12.0 mm to (44.9, 110.9), turned to -90 degrees
- moved C305 11.8 mm to (55.2, 129.8), turned to 0 degrees
- moved C307 11.7 mm to (57.5, 126.0), turned to -90 degrees
- moved R302 11.3 mm to (47.0, 112.5), turned to -90 degrees
- moved NT301 10.7 mm to (56.3, 127.9), turned to 180 degrees
- moved RE_ESP301 10.6 mm to (46.5, 101.5), turned to 180 degrees
- moved C301 9.28 mm to (44.9, 108.9), turned to 0 degrees
- moved R303 8.72 mm to (47.0, 110.6), turned to 90 degrees
- moved C306 7.61 mm to (55.2, 123.4), turned to 0 degrees
- moved IC301 7.44 mm to (55.1, 126.6), turned to 90 degrees
- moved J308 0.21 mm to (66.0, 136.7), turned to 0 degrees
- moved J305 0.21 mm to (66.0, 117.8), turned to 0 degrees
- moved Q302 0.21 mm to (62.6, 124.8)
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Connections:
- Q301 pad 1: IO14 -> IO48
- Q302 pad 1: IO12 -> IO34
- Q303 pad 1: IO13 -> IO33
- Q304 pad 1: IO15 -> IO47
- R304 pad 1: IO14 -> IO48
- R305 pad 1: IO12 -> IO34
- R306 pad 1: IO13 -> IO33
- R307 pad 1: IO15 -> IO47
- U303 pad 25: unconnected-(U303-IO21-Pad25) -> IO21
- U303 pad 26: unconnected-(U303-IO26-Pad26) -> IO26
- U303 pad 27: unconnected-(U303-IO47-Pad27) -> IO47
- U303 pad 28: unconnected-(U303-IO33-Pad28) -> IO33
- U303 pad 29: unconnected-(U303-IO34-Pad29) -> IO34
- U303 pad 30: unconnected-(U303-IO48-Pad30) -> IO48
- U303 pad 31: unconnected-(U303-IO35-Pad31) -> IO35
- U303 pad 32: unconnected-(U303-IO36-Pad32) -> IO36
- U303 pad 33: unconnected-(U303-IO37-Pad33) -> IO37
- U303 pad 34: unconnected-(U303-IO38-Pad34) -> IO38
- U303 pad 35: unconnected-(U303-IO39-Pad35) -> IO39
- U303 pad 36: unconnected-(U303-IO40-Pad36) -> IO40
- U303 pad 37: unconnected-(U303-IO41-Pad37) -> IO41
- U303 pad 38: unconnected-(U303-IO42-Pad38) -> IO42
- U303 pad 41: unconnected-(U303-IO45-Pad41) -> IO45
- U303 pad 44: unconnected-(U303-IO46-Pad44) -> IO46
Routing:
- net Net-(U303-EN): track 5.01 -> 18.1 mm, vias 1 -> 2
- net SCL: track 12.6 -> 2.72 mm, vias 1 -> 0
- net SDA: track 11.2 -> 2.71 mm, vias 1 -> 0
- net BOOT: track 1.65 -> 4.76 mm
- net GND: track 16.6 -> 14.4 mm, vias 8 -> 11
- net +3V3: track 72.1 -> 71.4 mm, vias 9 -> 8
- added copper zone on B.Cu, net VCC

Commit message: Connected IO
Parts:
- added NT601: NetTie_2, NetTie:NetTie-2_SMD_Pad0.5mm, F.Cu at (56.2, 138.9)
- added R_Sense601: 1, Resistor_SMD:R_0805_2012Metric, F.Cu at (58.1, 138.9)
- moved J310 12.4 mm to (45.9, 130.0)
- moved R310 12.4 mm to (48.5, 129.7)
- moved R311 12.4 mm to (48.5, 132.7)
- moved R312 12.4 mm to (48.5, 117.1)
- moved R313 12.4 mm to (48.5, 120.2)
- moved R314 12.4 mm to (48.5, 123.4)
- moved R315 12.4 mm to (48.5, 126.5)
- moved J311 12.4 mm to (45.9, 117.4)
- moved J312 12.4 mm to (45.9, 123.7)
- moved J303 3.30 mm to (53.1, 142.0)
- moved J304 3.30 mm to (58.1, 142.0)
- moved RE_ESP301 0.55 mm to (47.0, 101.7), turned to 90 degrees
- moved J301 0.51 mm to (44.4, 102.3)
- moved C301 0.10 mm to (45.0, 108.9)
- moved R301 0.10 mm to (45.4, 112.8)
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Connections:
- J304 pad 1: GND -> GND1
- R310 pad 2: IO17 -> IO14
- R311 pad 1: IO17 -> IO14
- R312 pad 2: IO18 -> IO12
- R313 pad 1: IO18 -> IO12
- R314 pad 2: IO11 -> IO13
- R315 pad 1: IO11 -> IO13
- U303 pad 6: unconnected-(U303-IO2-Pad6) -> IO2
Routing:
- net IO47: track 0.00 -> 27.9 mm, vias 0 -> 2
- net IO18: track 1.36 -> 24.6 mm, vias 0 -> 2
- net IO33: track 0.00 -> 22.6 mm, vias 0 -> 2
- net IO14: track 0.00 -> 18.9 mm
- net IO34: track 0.00 -> 12.6 mm
- net IO13: track 0.00 -> 11.9 mm
- net IO48: track 0.00 -> 6.23 mm
- net IO12: track 0.00 -> 5.56 mm
- net VCC: track 4.05 -> 6.05 mm
- net Net-(U303-EN): track 18.1 -> 16.5 mm
- net IO11: track 1.45 -> 0.00 mm
- net +3V3: track 71.4 -> 70.1 mm
- net IO17: track 1.35 -> 0.00 mm
- added copper zone on F.Cu, net GND1
- added copper zone on B.Cu, net IO18
- added copper zone on F.Cu, net IO18
- added copper zone on F.Cu, net IO33
- added copper zone on F.Cu, net IO34
- added copper zone on F.Cu, net IO47
- added copper zone on F.Cu, net IO48
- removed copper zone on F.Cu, net IO12
- removed copper zone on F.Cu, net IO13
- removed copper zone on F.Cu, net IO14
- removed copper zone on F.Cu, net IO15
Other:
- board size 28.1 x 47.2 mm -> 27 x 45.5 mm
- board text added: "IO33"
- board text added: "IO34"
- board text added: "IO47"
- board text added: "IO48"
- board text removed: "IO12"
- board text removed: "IO13"
- board text removed: "IO14"
- board text removed: "IO15"
