File: ESP32_RemoteWetherstation/Hardware/ESP32_RemoteWetherstation/IO.kicad_sch (KiCad schematic)
At the start: 0 parts

Commit message: placed all comps onesided (#11)
Changed lines of the file:
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@@
-		)
-	)
-	(global_label "IO14"
-		(shape input)
-		(at 31.75 30.48 180)
-		(fields_autoplaced yes)
-		(effects
-			(font
-				(size 1.27 1.27)
-			)
-			(justify right)
-		)
-		(property "Intersheetrefs" "${INTERSHEET_REFS}"
-			(at 24.4105 30.48 0)
-			(effects
-				(font
-					(size 1.27 1.27)
-				)
-				(justify right)
-				(hide yes)
-			)
-		)
-	)
-	(global_label "IO15"
-		(shape input)
-		(at 31.75 64.77 180)
-		(fields_autoplaced yes)
-		(effects
-			(font
-				(size 1.27 1.27)
-			)
-			(justify right)
-		)
-		(property "Intersheetrefs" "${INTERSHEET_REFS}"
-			(at 24.4105 64.77 0)
-			(effects
-				(font
-					(size 1.27 1.27)
-				)
-				(justify right)
-				(hide yes)
-			)
 		)
 	)
@@
 		)
 	)
-	(global_label "IO12"
+	(global_label "IO48"
+		(shape input)
+		(at 31.75 30.48 180)
+		(fields_autoplaced yes)
+		(effects
+			(font
+				(size 1.27 1.27)
+			)
+			(justify right)
+		)
+		(property "Intersheetrefs" "${INTERSHEET_REFS}"
+			(at 24.4105 30.48 0)
+			(effects
+				(font
+					(size 1.27 1.27)
+				)
+				(justify right)
+				(hide yes)
+			)
+		)
+	)
+	(global_label "IO34"
 		(shape input)
 		(at 31.75 41.91 180)
@@
 		(property "Intersheetrefs" "${INTERSHEET_REFS}"
 			(at 24.4105 41.91 0)
+			(effects
+				(font
+					(size 1.27 1.27)
+				)
+				(justify right)
+				(hide yes)
+			)
+		)
+	)
+	(global_label "IO47"
+		(shape input)
+		(at 31.75 64.77 180)
+		(fields_autoplaced yes)
+		(effects
+			(font
+				(size 1.27 1.27)
+			)
+			(justify right)
+		)
+		(property "Intersheetrefs" "${INTERSHEET_REFS}"
+			(at 24.4105 64.77 0)
 			(effects
 				(font
@@
 		)
 	)
-	(global_label "IO13"
-		(shape input)
-		(at 31.75 53.34 180)
-		(fields_autoplaced yes)
-		(effects
-			(font
-				(size 1.27 1.27)
-			)
-			(justify right)
-		)
-		(property "Intersheetrefs" "${INTERSHEET_REFS}"
-			(at 24.4105 53.34 0)
-			(effects
-				(font
-					(size 1.27 1.27)
-				)
-				(justify right)
-				(hide yes)
-			)
-		)
-	)
 	(global_label "IO17"
 		(shape input)
@@
 			(effects
 				(font
+					(size 1.27 1.27)
+				)
+				(justify right)
+				(hide yes)
+			)
+		)
+	)
+	(global_label "IO33"
+		(shape input)
+		(at 31.75 53.34 180)
+		(fields_autoplaced yes)
+		(effects
+			(font
+				(size 1.27 1.27)
+			)
+			(justify right)
+		)
+		(property "Intersheetrefs" "${INTERSHEET_REFS}"
+			(at 24.4105 53.34 0)
+			(effects
+				(font

Commit message: Connected IO
Changed lines of the file:
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@@
 		)
 	)
-	(global_label "IO18"
+	(global_label "IO13"
 		(shape input)
-		(at 93.98 40.64 180)
+		(at 93.98 52.07 180)
 		(fields_autoplaced yes)
 		(effects
@@
 		)
 		(property "Intersheetrefs" "${INTERSHEET_REFS}"
-			(at 86.6405 40.64 0)
+			(at 86.6405 52.07 0)
 			(effects
 				(font
@@
 		)
 	)
-	(global_label "IO11"
+	(global_label "IO12"
 		(shape input)
-		(at 93.98 52.07 180)
+		(at 93.98 40.64 180)
 		(fields_autoplaced yes)
 		(effects
@@
 		)
 		(property "Intersheetrefs" "${INTERSHEET_REFS}"
-			(at 86.6405 52.07 0)
+			(at 86.6405 40.64 0)
 			(effects
 				(font
@@
 		)
 	)
-	(global_label "IO17"
+	(global_label "IO14"
 		(shape input)
 		(at 93.98 29.21 180)
